Commit message: with the ceiling

File: src/Universal_Robots_ROS2_Tutorials/my_robot_cell/my_robot_cell_description/urdf/my_robot_cell_macro.xacro (robot description, xacro)
@@ -2,6 +2,6 @@
 <robot xmlns:xacro="http://ros.org/wiki/xacro">
   <xacro:include filename="$(find ur_description)/urdf/ur_macro.xacro"/>
+  <xacro:include filename="$(find my_robot_cell_description)/urdf/safety_wall.xacro"/>
   <xacro:include filename="$(find my_robot_cell_description)/urdf/table.xacro"/>
-  <xacro:include filename="$(find my_robot_cell_description)/urdf/safety_wall.xacro"/>
   <xacro:macro name="my_robot_cell" params="
     parent
@@ -21,7 +21,7 @@
     <link name="robot_mount"/>
     <joint name="base_to_robot_mount" type="fixed">
-      <parent link="table"/>
+      <parent link="robot_base_plate"/>
       <child link="robot_mount"/>
-      <origin xyz="-0.52 0.32 0" rpy="0 0 ${pi}" />
+      <origin xyz="0 0 0" rpy="0 0 ${pi}" />
     </joint>
     <!--This will create the specific robot-->

File: src/Universal_Robots_ROS2_Tutorials/my_robot_cell/my_robot_cell_description/urdf/safety_wall.xacro (robot description, xacro)
@@ -6,20 +6,27 @@
       <parent link="world"/>
       <child link="wall_wall_wall"/>
-      <origin xyz="0 0.505 1.25"/>
+      <origin xyz="0 0.505 1.2"/>
     </joint>
     <link name="wall_wall_wall">
       <visual>
         <geometry>
-          <box size="2.02 0.01 2.5"/>
+          <box size="2.02 0.01 2.4"/>
         </geometry>
-        <material name="gray">
-          <color rgba="0.5 0.5 0.5 1.0"/>
+        <material name="white">
+          <color rgba= "1 1 1 1"/>
         </material>
       </visual>
       <collision>
         <geometry>
-          <box size="2.02 0.01 2.5"/>
+          <box size="2.02 0.01 2.4"/>
         </geometry>
       </collision>
+      <inertial>
+      <mass value="100.0"/>
+      <inertia
+        ixx="1.0" ixy="0.0" ixz="0.0"
+        iyy="1.0" iyz="0.0"
+        izz="1.0"/>
+    </inertial>
     </link>
     <!-- Wall_left -->
@@ -27,10 +34,10 @@
       <parent link="world"/>
       <child link="wall_left"/>
-      <origin xyz="-1.005 -0.15 1.25"/>
+      <origin xyz="-1.005 -0.15 1.2"/>
     </joint>
     <link name="wall_left">
       <visual>
         <geometry>
-          <box size="0.01 1.3 2.5"/>
+          <box size="0.01 1.3 2.4"/>
         </geometry>
         <material name="see-through">
@@ -40,5 +47,5 @@
       <collision>
         <geometry>
-          <box size="0.01 1.2999 2.5"/>
+          <box size="0.01 1.2999 2.4"/>
         </geometry>
       </collision>
@@ -48,10 +55,10 @@
       <parent link="world"/>
       <child link="wall_right"/>
-      <origin xyz="1.005 -0.15 1.25"/>
+      <origin xyz="1.005 -0.15 1.2"/>
     </joint>
     <link name="wall_right">
       <visual>
         <geometry>
-          <box size="0.01 1.3 2.5"/>
+          <box size="0.01 1.3 2.4"/>
         </geometry>
         <material name="see-through">
@@ -61,5 +68,5 @@
       <collision>
         <geometry>
-          <box size="0.01 1.2999 2.5"/>
+          <box size="0.01 1.2999 2.4"/>
         </geometry>
       </collision>
@@ -69,10 +76,10 @@
       <parent link="world"/>
       <child link="wall_front"/>
-      <origin xyz="0 -0.805 1.25"/>
+      <origin xyz="0 -0.805 1.2"/>
     </joint>
     <link name="wall_front">
       <visual>
         <geometry>
-          <box size="2.02 0.01 2.5"/>
+          <box size="2.02 0.01 2.4"/>
         </geometry>
         <material name="see-through">
@@ -82,5 +89,26 @@
       <collision>
         <geometry>
-          <box size="2.02 0.01 2.5"/>
+          <box size="2.02 0.01 2.4"/>
+        </geometry>
+      </collision>
+    </link>
+    <!-- wall_ceiling -->
+    <joint name="base_to_wall_ceiling" type="fixed">
+      <parent link="world"/>
+      <child link="wall_ceiling"/>
+      <origin xyz="0 -0.15 2.405"/>
+    </joint>
+    <link name="wall_ceiling">
+      <visual>
+        <geometry>
+          <box size="2.02 1.32 0.01"/>
+        </geometry>
+        <material name="see-through">
+          <color rgba="0.5 0.5 0.5 0.1"/>
+        </material>
+      </visual>
+      <collision>
+        <geometry>
+          <box size="2.02 1.32 0.0099"/>
         </geometry>
       </collision>

File: src/Universal_Robots_ROS2_Tutorials/my_robot_cell/my_robot_cell_description/urdf/table.xacro (robot description, xacro)
@@ -3,7 +3,7 @@
   <xacro:macro name="table" params="parent *origin">
     <joint name="table_base_joint" type="fixed">
-      <xacro:insert_block name="origin"/>
       <parent link="${parent}" />
       <child link="table" />
+      <origin rpy="0 0 0" xyz="0 0 0.9"/>
     </joint>
     <link name="table">
@@ -31,4 +31,33 @@
       </inertial>
     </link>
+    <joint name="robot_base_plate_joint" type="fixed">
+      <parent link="table" />
+      <child link="robot_base_plate"/>
+      <origin rpy="0 0 0" xyz="-0.52 0.32 0.02"/>
+    </joint>
+    <link name="robot_base_plate">
+      <visual>
+        <geometry>
+          <box size="0.16 0.16 0.02"/>
+        </geometry>
+        <origin xyz= "0 0 -0.01"/>
+        <material name="grey">
+          <color rgba="0.5 0.5 0.5 1.0"/>
+        </material>
+      </visual>
+      <collision>
+        <geometry>
+          <box size="0.16 0.16 0.01999"/>
+        </geometry>
+        <origin xyz= "0 0 -0.01"/>
+      </collision>
+      <inertial>
+        <mass value="2.0"/>
+        <inertia
+        ixx="1.0" ixy="0.0" ixz="0.0"
+        iyy="1.0" iyz="0.0"
+        izz="1.0"/>
+      </inertial>
+    </link>
   </xacro:macro>
 </robot>

Commit message: with gripper attached no moveit!

File: src/Universal_Robots_ROS2_Tutorials/my_robot_cell/my_robot_cell_description/urdf/my_robot_cell_macro.xacro (robot description, xacro)
@@ -4,4 +4,5 @@
   <xacro:include filename="$(find my_robot_cell_description)/urdf/safety_wall.xacro"/>
   <xacro:include filename="$(find my_robot_cell_description)/urdf/table.xacro"/>
+  <xacro:include filename="$(find my_robot_cell_description)/urdf/2fg7_gripper/urdf/onrobot_2fg7_gripper.urdf.xacro"/>
   <xacro:macro name="my_robot_cell" params="
     parent
@@ -37,4 +38,7 @@
       <origin xyz="0 0 0" rpy="0 0 0" />
     </xacro:ur_robot>
+    <xacro:onrobot_2fg7_gripper prefix="onrobot_2fg7_gripper" parent ="ur5e_tool0">
+      <origin rpy="0 4.71239 0" xyz="0 0 0"/>
+    </xacro:onrobot_2fg7_gripper>
   </xacro:macro>
 </robot>

Commit message: with box as gripper

File: src/Universal_Robots_ROS2_Tutorials/my_robot_cell/my_robot_cell_description/urdf/my_robot_cell_macro.xacro (robot description, xacro)
@@ -5,4 +5,5 @@
   <xacro:include filename="$(find my_robot_cell_description)/urdf/table.xacro"/>
   <xacro:include filename="$(find my_robot_cell_description)/urdf/2fg7_gripper/urdf/onrobot_2fg7_gripper.urdf.xacro"/>
+  <xacro:include filename="$(find my_robot_cell_description)/urdf/box.xacro"/>
   <xacro:macro name="my_robot_cell" params="
     parent
@@ -38,7 +39,10 @@
       <origin xyz="0 0 0" rpy="0 0 0" />
     </xacro:ur_robot>
-    <xacro:onrobot_2fg7_gripper prefix="onrobot_2fg7_gripper" parent ="ur5e_tool0">
+    <xacro:box parent="ur5e_tool0">
+      <origin xyz="0 0 0.1" rpy="0 0 0"/>
+    </xacro:box>
+    <!--xacro:onrobot_2fg7_gripper prefix="onrobot_2fg7_gripper" parent ="ur5e_tool0">
       <origin rpy="0 4.71239 0" xyz="0 0 0"/>
-    </xacro:onrobot_2fg7_gripper>
+    </xacro:onrobot_2fg7_gripper-->
   </xacro:macro>
 </robot>

Commit message: with second robot plate

File: src/Universal_Robots_ROS2_Tutorials/my_robot_cell/my_robot_cell_description/urdf/my_robot_cell_macro.xacro (robot description, xacro)
@@ -22,6 +22,6 @@
     </xacro:safety_wall>
     <link name="robot_mount"/>
-    <joint name="base_to_robot_mount" type="fixed">
-      <parent link="robot_base_plate"/>
+    <joint name="base_to_robot_mount_409" type="fixed">
+      <parent link="robot_base_plate_409"/>
       <child link="robot_mount"/>
       <origin xyz="0 0 0" rpy="0 0 ${pi}" />

File: src/Universal_Robots_ROS2_Tutorials/my_robot_cell/my_robot_cell_description/urdf/table.xacro (robot description, xacro)
@@ -31,10 +31,41 @@
       </inertial>
     </link>
-    <joint name="robot_base_plate_joint" type="fixed">
+    <!--For Robot 409-->
+    <joint name="robot_base_plate_joint_409" type="fixed">
       <parent link="table" />
-      <child link="robot_base_plate"/>
+      <child link="robot_base_plate_409"/>
       <origin rpy="0 0 0" xyz="-0.52 0.32 0.02"/>
     </joint>
-    <link name="robot_base_plate">
+    <link name="robot_base_plate_409">
+      <visual>
+        <geometry>
+          <box size="0.16 0.16 0.02"/>
+        </geometry>
+        <origin xyz= "0 0 -0.01"/>
+        <material name="grey">
+          <color rgba="0.5 0.5 0.5 1.0"/>
+        </material>
+      </visual>
+      <collision>
+        <geometry>
+          <box size="0.16 0.16 0.01999"/>
+        </geometry>
+        <origin xyz= "0 0 -0.01"/>
+      </collision>
+      <inertial>
+        <mass value="2.0"/>
+        <inertia
+        ixx="1.0" ixy="0.0" ixz="0.0"
+        iyy="1.0" iyz="0.0"
+        izz="1.0"/>
+      </inertial>
+    </link>
+    <!--For Robot 410-->
+    <joint name="robot_base_plate_joint_410" type="fixed">
+      <parent link="table" />
+      <child link="robot_base_plate_410"/>
+      <origin rpy="0 0 0" xyz="0.52 -0.32 0.02"/>
+    </joint>
+    <link name="robot_base_plate_410">
       <visual>
         <geometry>
