Commit message: with box parametrized

File: src/Universal_Robots_ROS2_Tutorials/my_robot_cell/my_robot_cell_description/urdf/box.xacro (robot description, xacro)
@@ -1,11 +1,11 @@
 <?xml version="1.0"?>
 <robot xmlns:xacro="http://ros.org/wiki/xacro">
-  <xacro:macro name="box" params="parent *origin">
-    <joint name="409_box_joint" type="fixed">
-      <parent link="409_ur5e_tool0" />
-      <child link="box" />
+  <xacro:macro name="box" params="parent prefix *origin">
+    <joint name="${prefix}_box_joint" type="fixed">
+      <parent link="${prefix}_ur5e_tool0" />
+      <child link="${prefix}_box" />
       <origin rpy="0 0 0" xyz="0 0 0.16"/>
     </joint>
-    <link name="box">
+    <link name="${prefix}_box">
       <visual>
         <geometry>

File: src/Universal_Robots_ROS2_Tutorials/my_robot_cell/my_robot_cell_description/urdf/my_robot_cell_macro.xacro (robot description, xacro)
@@ -32,5 +32,5 @@
       <origin xyz="0 0 0" rpy="0 0 0" />
     </xacro:ur_robot>
-    <xacro:box parent="${prefix}_ur5e_tool0">
+    <xacro:box parent="${prefix}_ur5e_tool0" prefix="${prefix}">
       <origin xyz="0 0 0.1" rpy="0 0 0"/>
     </xacro:box>

File: src/Universal_Robots_ROS2_Tutorials/my_robot_cell/my_robot_cell_description/urdf/table.xacro (robot description, xacro)
@@ -60,4 +60,33 @@
       </inertial>
     </link>
+    <joint name="410_robot_base_plate_joint" type="fixed">
+      <parent link="table" />
+      <child link="410_robot_base_plate"/>
+      <origin rpy="0 0 0" xyz="0.52 -0.32 0.02"/>
+    </joint>
+    <link name="410_robot_base_plate">
+      <visual>
+        <geometry>
+          <box size="0.16 0.16 0.02"/>
+        </geometry>
+        <origin xyz= "0 0 -0.01"/>
+        <material name="grey">
+          <color rgba="0.5 0.5 0.5 1.0"/>
+        </material>
+      </visual>
+      <collision>
+        <geometry>
+          <box size="0.16 0.16 0.01999"/>
+        </geometry>
+        <origin xyz= "0 0 -0.01"/>
+      </collision>
+      <inertial>
+        <mass value="2.0"/>
+        <inertia
+        ixx="1.0" ixy="0.0" ixz="0.0"
+        iyy="1.0" iyz="0.0"
+        izz="1.0"/>
+      </inertial>
+    </link>
   </xacro:macro>
 </robot>
