Commit message: with robot one name 409

File: src/Universal_Robots_ROS2_Tutorials/my_robot_cell/moveit_config/config/my_robot_cell.ros2_control.xacro (robot description, xacro)
@@ -8,49 +8,49 @@
                 <plugin>mock_components/GenericSystem</plugin>
             </hardware>
-            <joint name="ur5e_shoulder_pan_joint">
+            <joint name="ur5e_409_shoulder_pan_joint">
                 <command_interface name="position"/>
                 <command_interface name="velocity"/>
                 <state_interface name="position">
-                  <param name="initial_value">${initial_positions['ur5e_shoulder_pan_joint']}</param>
+                  <param name="initial_value">${initial_positions['ur5e_409_shoulder_pan_joint']}</param>
                 </state_interface>
                 <state_interface name="velocity"/>
             </joint>
-            <joint name="ur5e_shoulder_lift_joint">
+            <joint name="ur5e_409_shoulder_lift_joint">
                 <command_interface name="position"/>
                 <command_interface name="velocity"/>
                 <state_interface name="position">
-                  <param name="initial_value">${initial_positions['ur5e_shoulder_lift_joint']}</param>
+                  <param name="initial_value">${initial_positions['ur5e_409_shoulder_lift_joint']}</param>
                 </state_interface>
                 <state_interface name="velocity"/>
             </joint>
-            <joint name="ur5e_elbow_joint">
+            <joint name="ur5e_409_elbow_joint">
                 <command_interface name="position"/>
                 <command_interface name="velocity"/>
                 <state_interface name="position">
-                  <param name="initial_value">${initial_positions['ur5e_elbow_joint']}</param>
+                  <param name="initial_value">${initial_positions['ur5e_409_elbow_joint']}</param>
                 </state_interface>
                 <state_interface name="velocity"/>
             </joint>
-            <joint name="ur5e_wrist_1_joint">
+            <joint name="ur5e_409_wrist_1_joint">
                 <command_interface name="position"/>
                 <command_interface name="velocity"/>
                 <state_interface name="position">
-                  <param name="initial_value">${initial_positions['ur5e_wrist_1_joint']}</param>
+                  <param name="initial_value">${initial_positions['ur5e_409_wrist_1_joint']}</param>
                 </state_interface>
                 <state_interface name="velocity"/>
             </joint>
-            <joint name="ur5e_wrist_2_joint">
+            <joint name="ur5e_409_wrist_2_joint">
                 <command_interface name="position"/>
                 <command_interface name="velocity"/>
                 <state_interface name="position">
-                  <param name="initial_value">${initial_positions['ur5e_wrist_2_joint']}</param>
+                  <param name="initial_value">${initial_positions['ur5e_409_wrist_2_joint']}</param>
                 </state_interface>
                 <state_interface name="velocity"/>
             </joint>
-            <joint name="ur5e_wrist_3_joint">
+            <joint name="ur5e_409_wrist_3_joint">
                 <command_interface name="position"/>
                 <command_interface name="velocity"/>
                 <state_interface name="position">
-                  <param name="initial_value">${initial_positions['ur5e_wrist_3_joint']}</param>
+                  <param name="initial_value">${initial_positions['ur5e_409_wrist_3_joint']}</param>
                 </state_interface>
                 <state_interface name="velocity"/>

File: src/Universal_Robots_ROS2_Tutorials/my_robot_cell/my_robot_cell_control/urdf/my_robot_cell_controlled.urdf.xacro (robot description, xacro)
@@ -33,5 +33,5 @@
   <xacro:ur_ros2_control
     name="$(arg ur_type)"
-    tf_prefix="$(arg ur_type)_"
+    tf_prefix="ur5e_409_"
     kinematics_parameters_file="$(arg kinematics_parameters_file)"
     robot_ip="$(arg robot_ip)"

File: src/Universal_Robots_ROS2_Tutorials/my_robot_cell/my_robot_cell_description/urdf/box.xacro (robot description, xacro)
@@ -3,5 +3,5 @@
   <xacro:macro name="box" params="parent *origin">
     <joint name="box_joint" type="fixed">
-      <parent link="ur5e_tool0" />
+      <parent link="ur5e_409_tool0" />
       <child link="box" />
       <origin rpy="0 0 0" xyz="0 0 0.16"/>

File: src/Universal_Robots_ROS2_Tutorials/my_robot_cell/my_robot_cell_description/urdf/my_robot_cell_macro.xacro (robot description, xacro)
@@ -29,6 +29,6 @@
     <!--This will create the specific robot-->
     <xacro:ur_robot
-      name="${ur_type}"
-      tf_prefix="${ur_type}_"
+      name="${ur_type}_409"
+      tf_prefix="${ur_type}_409_"
       parent="robot_mount"
       joint_limits_parameters_file="${joint_limits_parameters_file}"
@@ -39,5 +39,5 @@
       <origin xyz="0 0 0" rpy="0 0 0" />
     </xacro:ur_robot>
-    <xacro:box parent="ur5e_tool0">
+    <xacro:box parent="ur5e_409_tool0">
       <origin xyz="0 0 0.1" rpy="0 0 0"/>
     </xacro:box>

Commit message: with one robot, new start because other failed

File: src/Universal_Robots_ROS2_Tutorials/my_robot_cell/moveit_config/config/my_robot_cell.ros2_control.xacro (robot description, xacro)
@@ -8,49 +8,49 @@
                 <plugin>mock_components/GenericSystem</plugin>
             </hardware>
-            <joint name="ur5e_409_shoulder_pan_joint">
+            <joint name="ur5e_shoulder_pan_joint">
                 <command_interface name="position"/>
                 <command_interface name="velocity"/>
                 <state_interface name="position">
-                  <param name="initial_value">${initial_positions['ur5e_409_shoulder_pan_joint']}</param>
+                  <param name="initial_value">${initial_positions['ur5e_shoulder_pan_joint']}</param>
                 </state_interface>
                 <state_interface name="velocity"/>
             </joint>
-            <joint name="ur5e_409_shoulder_lift_joint">
+            <joint name="ur5e_shoulder_lift_joint">
                 <command_interface name="position"/>
                 <command_interface name="velocity"/>
                 <state_interface name="position">
-                  <param name="initial_value">${initial_positions['ur5e_409_shoulder_lift_joint']}</param>
+                  <param name="initial_value">${initial_positions['ur5e_shoulder_lift_joint']}</param>
                 </state_interface>
                 <state_interface name="velocity"/>
             </joint>
-            <joint name="ur5e_409_elbow_joint">
+            <joint name="ur5e_elbow_joint">
                 <command_interface name="position"/>
                 <command_interface name="velocity"/>
                 <state_interface name="position">
-                  <param name="initial_value">${initial_positions['ur5e_409_elbow_joint']}</param>
+                  <param name="initial_value">${initial_positions['ur5e_elbow_joint']}</param>
                 </state_interface>
                 <state_interface name="velocity"/>
             </joint>
-            <joint name="ur5e_409_wrist_1_joint">
+            <joint name="ur5e_wrist_1_joint">
                 <command_interface name="position"/>
                 <command_interface name="velocity"/>
                 <state_interface name="position">
-                  <param name="initial_value">${initial_positions['ur5e_409_wrist_1_joint']}</param>
+                  <param name="initial_value">${initial_positions['ur5e_wrist_1_joint']}</param>
                 </state_interface>
                 <state_interface name="velocity"/>
             </joint>
-            <joint name="ur5e_409_wrist_2_joint">
+            <joint name="ur5e_wrist_2_joint">
                 <command_interface name="position"/>
                 <command_interface name="velocity"/>
                 <state_interface name="position">
-                  <param name="initial_value">${initial_positions['ur5e_409_wrist_2_joint']}</param>
+                  <param name="initial_value">${initial_positions['ur5e_wrist_2_joint']}</param>
                 </state_interface>
                 <state_interface name="velocity"/>
             </joint>
-            <joint name="ur5e_409_wrist_3_joint">
+            <joint name="ur5e_wrist_3_joint">
                 <command_interface name="position"/>
                 <command_interface name="velocity"/>
                 <state_interface name="position">
-                  <param name="initial_value">${initial_positions['ur5e_409_wrist_3_joint']}</param>
+                  <param name="initial_value">${initial_positions['ur5e_wrist_3_joint']}</param>
                 </state_interface>
                 <state_interface name="velocity"/>

File: src/Universal_Robots_ROS2_Tutorials/my_robot_cell/my_robot_cell_control/urdf/my_robot_cell_controlled.urdf.xacro (robot description, xacro)
@@ -5,6 +5,4 @@
   <!--The driver already provides a control tag for the UR arm, we can directly include-->
   <xacro:include filename="$(find ur_robot_driver)/urdf/ur.ros2_control.xacro"/>
-  <xacro:include filename="$(find my_robot_cell_description)/urdf/safety_wall.xacro"/>
-  <xacro:include filename="$(find my_robot_cell_description)/urdf/table.xacro"/>
   <!--We need to specify the arguments used for parametrizing our description-->
   <xacro:arg name="ur_type" default="ur5e"/>
@@ -22,10 +20,4 @@
   <link name="world" />
   <!--Create the scene description including the robot-->
-  <xacro:safety_wall parent="world">
-    <origin rpy="0 0 0" xyz="0 0 0"/>
-  </xacro:safety_wall>
-  <xacro:table parent="world">
-    <origin rpy="0 0 0" xyz="0 -0 0.9"/>
-  </xacro:table>
   <xacro:my_robot_cell
     parent="world"
@@ -41,5 +33,5 @@
   <xacro:ur_ros2_control
     name="$(arg ur_type)"
-    tf_prefix="ur5e_409_"
+    tf_prefix="$(arg ur_type)_"
     kinematics_parameters_file="$(arg kinematics_parameters_file)"
     robot_ip="$(arg robot_ip)"

File: src/Universal_Robots_ROS2_Tutorials/my_robot_cell/my_robot_cell_description/urdf/box.xacro (robot description, xacro)
@@ -3,5 +3,5 @@
   <xacro:macro name="box" params="parent *origin">
     <joint name="box_joint" type="fixed">
-      <parent link="ur5e_409_tool0" />
+      <parent link="ur5e_tool0" />
       <child link="box" />
       <origin rpy="0 0 0" xyz="0 0 0.16"/>

File: src/Universal_Robots_ROS2_Tutorials/my_robot_cell/my_robot_cell_description/urdf/my_robot_cell.urdf.xacro (robot description, xacro)
@@ -2,6 +2,4 @@
 <robot name="my_robot_cell" xmlns:xacro="http://ros.org/wiki/xacro">
   <xacro:include filename="$(find my_robot_cell_description)/urdf/my_robot_cell_macro.xacro"/>
-  <xacro:include filename="$(find my_robot_cell_description)/urdf/safety_wall.xacro"/>
-  <xacro:include filename="$(find my_robot_cell_description)/urdf/table.xacro"/>
   <xacro:arg name="ur_type" default="ur5e"/>
   <xacro:arg name="joint_limits_parameters_file" default="$(find ur_description)/config/$(arg ur_type)/joint_limits.yaml"/>
@@ -11,14 +9,7 @@
   <link name="world"/>
   <!--This will create the scene where the robot is located in-->
-  <xacro:safety_wall parent="world">
-    <origin rpy="0 0 0" xyz="0 0 0"/>
-  </xacro:safety_wall>
-  <xacro:table parent="world">
-    <origin rpy="0 0 0" xyz="0 -0 0.9"/>
-  </xacro:table>
   <xacro:my_robot_cell
     parent="world"
     ur_type="$(arg ur_type)"
-    prefix="409"
     joint_limits_parameters_file="$(arg joint_limits_parameters_file)"
     kinematics_parameters_file="$(arg kinematics_parameters_file)"

File: src/Universal_Robots_ROS2_Tutorials/my_robot_cell/my_robot_cell_description/urdf/my_robot_cell_macro.xacro (robot description, xacro)
@@ -2,4 +2,6 @@
 <robot xmlns:xacro="http://ros.org/wiki/xacro">
   <xacro:include filename="$(find ur_description)/urdf/ur_macro.xacro"/>
+  <xacro:include filename="$(find my_robot_cell_description)/urdf/safety_wall.xacro"/>
+  <xacro:include filename="$(find my_robot_cell_description)/urdf/table.xacro"/>
   <xacro:include filename="$(find my_robot_cell_description)/urdf/box.xacro"/>
   <xacro:include filename="$(find my_robot_cell_description)/urdf/2fg7_gripper/urdf/onrobot_2fg7_gripper.urdf.xacro"/>
@@ -13,4 +15,10 @@
     visual_parameters_file
     ">
+    <xacro:table parent="${parent}">
+      <origin rpy="0 0 0" xyz="0 -0 0.9"/>
+    </xacro:table>
+    <xacro:safety_wall parent="${parent}">
+      <origin rpy="0 0 0" xyz="0 0 0"/>
+    </xacro:safety_wall>
     <link name="robot_mount"/>
     <joint name="base_to_robot_mount" type="fixed">
@@ -21,6 +29,6 @@
     <!--This will create the specific robot-->
     <xacro:ur_robot
-      name="${ur_type}_409"
-      tf_prefix="${ur_type}_409_"
+      name="${ur_type}"
+      tf_prefix="${ur_type}_"
       parent="robot_mount"
       joint_limits_parameters_file="${joint_limits_parameters_file}"
@@ -31,5 +39,5 @@
       <origin xyz="0 0 0" rpy="0 0 0" />
     </xacro:ur_robot>
-    <xacro:box parent="ur5e_409_tool0">
+    <xacro:box parent="ur5e_tool0">
       <origin xyz="0 0 0.1" rpy="0 0 0"/>
     </xacro:box>

File: src/Universal_Robots_ROS2_Tutorials/my_robot_cell/my_robot_cell_description/urdf/table.xacro (robot description, xacro)
@@ -31,5 +31,4 @@
       </inertial>
     </link>
-    <!--For Robot 409-->
     <joint name="robot_base_plate_joint" type="fixed">
       <parent link="table" />
@@ -61,34 +60,4 @@
       </inertial>
     </link>
-    <!--For Robot 410-->
-    <joint name="robot_base_plate_joint_410" type="fixed">
-      <parent link="table" />
-      <child link="robot_base_plate_410"/>
-      <origin rpy="0 0 0" xyz="0.52 -0.32 0.02"/>
-    </joint>
-    <link name="robot_base_plate_410">
-      <visual>
-        <geometry>
-          <box size="0.16 0.16 0.02"/>
-        </geometry>
-        <origin xyz= "0 0 -0.01"/>
-        <material name="grey">
-          <color rgba="0.5 0.5 0.5 1.0"/>
-        </material>
-      </visual>
-      <collision>
-        <geometry>
-          <box size="0.16 0.16 0.01999"/>
-        </geometry>
-        <origin xyz= "0 0 -0.01"/>
-      </collision>
-      <inertial>
-        <mass value="2.0"/>
-        <inertia
-        ixx="1.0" ixy="0.0" ixz="0.0"
-        iyy="1.0" iyz="0.0"
-        izz="1.0"/>
-      </inertial>
-    </link>
   </xacro:macro>
 </robot>

Commit message: one robot fully parametrized and setup assistant still works

File: src/Universal_Robots_ROS2_Tutorials/my_robot_cell/moveit_config/config/my_robot_cell.ros2_control.xacro (robot description, xacro)
@@ -8,51 +8,63 @@
                 <plugin>mock_components/GenericSystem</plugin>
             </hardware>
-            <joint name="ur5e_shoulder_pan_joint">
+            <joint name="409_ur5e_shoulder_pan_joint">
                 <command_interface name="position"/>
                 <command_interface name="velocity"/>
+                <command_interface name="effort"/>
                 <state_interface name="position">
-                  <param name="initial_value">${initial_positions['ur5e_shoulder_pan_joint']}</param>
+                  <param name="initial_value">${initial_positions['409_ur5e_shoulder_pan_joint']}</param>
                 </state_interface>
                 <state_interface name="velocity"/>
+                <state_interface name="effort"/>
             </joint>
-            <joint name="ur5e_shoulder_lift_joint">
+            <joint name="409_ur5e_shoulder_lift_joint">
                 <command_interface name="position"/>
                 <command_interface name="velocity"/>
+                <command_interface name="effort"/>
                 <state_interface name="position">
-                  <param name="initial_value">${initial_positions['ur5e_shoulder_lift_joint']}</param>
+                  <param name="initial_value">${initial_positions['409_ur5e_shoulder_lift_joint']}</param>
                 </state_interface>
                 <state_interface name="velocity"/>
+                <state_interface name="effort"/>
             </joint>
-            <joint name="ur5e_elbow_joint">
+            <joint name="409_ur5e_elbow_joint">
                 <command_interface name="position"/>
                 <command_interface name="velocity"/>
+                <command_interface name="effort"/>
                 <state_interface name="position">
-                  <param name="initial_value">${initial_positions['ur5e_elbow_joint']}</param>
+                  <param name="initial_value">${initial_positions['409_ur5e_elbow_joint']}</param>
                 </state_interface>
                 <state_interface name="velocity"/>
+                <state_interface name="effort"/>
             </joint>
-            <joint name="ur5e_wrist_1_joint">
+            <joint name="409_ur5e_wrist_1_joint">
                 <command_interface name="position"/>
                 <command_interface name="velocity"/>
+                <command_interface name="effort"/>
                 <state_interface name="position">
-                  <param name="initial_value">${initial_positions['ur5e_wrist_1_joint']}</param>
+                  <param name="initial_value">${initial_positions['409_ur5e_wrist_1_joint']}</param>
                 </state_interface>
                 <state_interface name="velocity"/>
+                <state_interface name="effort"/>
             </joint>
-            <joint name="ur5e_wrist_2_joint">
+            <joint name="409_ur5e_wrist_2_joint">
                 <command_interface name="position"/>
                 <command_interface name="velocity"/>
+                <command_interface name="effort"/>
                 <state_interface name="position">
-                  <param name="initial_value">${initial_positions['ur5e_wrist_2_joint']}</param>
+                  <param name="initial_value">${initial_positions['409_ur5e_wrist_2_joint']}</param>
                 </state_interface>
                 <state_interface name="velocity"/>
+                <state_interface name="effort"/>
             </joint>
-            <joint name="ur5e_wrist_3_joint">
+            <joint name="409_ur5e_wrist_3_joint">
                 <command_interface name="position"/>
                 <command_interface name="velocity"/>
+                <command_interface name="effort"/>
                 <state_interface name="position">
-                  <param name="initial_value">${initial_positions['ur5e_wrist_3_joint']}</param>
+                  <param name="initial_value">${initial_positions['409_ur5e_wrist_3_joint']}</param>
                 </state_interface>
                 <state_interface name="velocity"/>
+                <state_interface name="effort"/>
             </joint>
         </ros2_control>

File: src/Universal_Robots_ROS2_Tutorials/my_robot_cell/my_robot_cell_control/urdf/my_robot_cell_controlled.urdf.xacro (robot description, xacro)
@@ -31,4 +31,5 @@
     parent="world"
     ur_type="$(arg ur_type)"
+    prefix="409"
     joint_limits_parameters_file="$(arg joint_limit_parameters_file)"
     kinematics_parameters_file="$(arg kinematics_parameters_file)"
@@ -41,5 +42,5 @@
   <xacro:ur_ros2_control
     name="$(arg ur_type)"
-    tf_prefix="$(arg ur_type)_"
+    tf_prefix="409_$(arg ur_type)_"
     kinematics_parameters_file="$(arg kinematics_parameters_file)"
     robot_ip="$(arg robot_ip)"

File: src/Universal_Robots_ROS2_Tutorials/my_robot_cell/my_robot_cell_description/urdf/box.xacro (robot description, xacro)
@@ -2,6 +2,6 @@
 <robot xmlns:xacro="http://ros.org/wiki/xacro">
   <xacro:macro name="box" params="parent *origin">
-    <joint name="box_joint" type="fixed">
-      <parent link="ur5e_tool0" />
+    <joint name="409_box_joint" type="fixed">
+      <parent link="409_ur5e_tool0" />
       <child link="box" />
       <origin rpy="0 0 0" xyz="0 0 0.16"/>

File: src/Universal_Robots_ROS2_Tutorials/my_robot_cell/my_robot_cell_description/urdf/my_robot_cell.urdf.xacro (robot description, xacro)
@@ -20,4 +20,5 @@
     parent="world"
     ur_type="$(arg ur_type)"
+    prefix="409"
     joint_limits_parameters_file="$(arg joint_limits_parameters_file)"
     kinematics_parameters_file="$(arg kinematics_parameters_file)"

File: src/Universal_Robots_ROS2_Tutorials/my_robot_cell/my_robot_cell_description/urdf/my_robot_cell_macro.xacro (robot description, xacro)
@@ -8,4 +8,5 @@
     *origin
     ur_type
+    prefix
     joint_limits_parameters_file
     kinematics_parameters_file
@@ -13,15 +14,15 @@
     visual_parameters_file
     ">
-    <link name="robot_mount"/>
-    <joint name="base_to_robot_mount" type="fixed">
-      <parent link="robot_base_plate"/>
-      <child link="robot_mount"/>
+    <link name="${prefix}_robot_mount"/>
+    <joint name="${prefix}_base_to_robot_mount" type="fixed">
+      <parent link="${prefix}_robot_base_plate"/>
+      <child link="${prefix}_robot_mount"/>
       <origin xyz="0 0 0" rpy="0 0 ${pi}" />
     </joint>
     <!--This will create the specific robot-->
     <xacro:ur_robot
-      name="${ur_type}"
-      tf_prefix="${ur_type}_"
-      parent="robot_mount"
+      name="${prefix}_${ur_type}"
+      tf_prefix="${prefix}_${ur_type}_"
+      parent="${prefix}_robot_mount"
       joint_limits_parameters_file="${joint_limits_parameters_file}"
       kinematics_parameters_file="${kinematics_parameters_file}"
@@ -31,5 +32,5 @@
       <origin xyz="0 0 0" rpy="0 0 0" />
     </xacro:ur_robot>
-    <xacro:box parent="ur5e_tool0">
+    <xacro:box parent="${prefix}_ur5e_tool0">
       <origin xyz="0 0 0.1" rpy="0 0 0"/>
     </xacro:box>

File: src/Universal_Robots_ROS2_Tutorials/my_robot_cell/my_robot_cell_description/urdf/table.xacro (robot description, xacro)
@@ -31,10 +31,10 @@
       </inertial>
     </link>
-    <joint name="robot_base_plate_joint" type="fixed">
+    <joint name="409_robot_base_plate_joint" type="fixed">
       <parent link="table" />
-      <child link="robot_base_plate"/>
+      <child link="409_robot_base_plate"/>
       <origin rpy="0 0 0" xyz="-0.52 0.32 0.02"/>
     </joint>
-    <link name="robot_base_plate">
+    <link name="409_robot_base_plate">
       <visual>
         <geometry>
