Commit message: motion planning running with two robots but still some small errors

File: src/Universal_Robots_ROS2_Tutorials/my_robot_cell/moveit_config/config/my_robot_cell.ros2_control.xacro (robot description, xacro)
@@ -68,4 +68,64 @@
                 <state_interface name="effort"/>
             </joint>
+            <joint name="410_ur5e_shoulder_pan_joint">
+                <command_interface name="position"/>
+                <command_interface name="velocity"/>
+                <command_interface name="effort"/>
+                <state_interface name="position">
+                  <param name="initial_value">${initial_positions['410_ur5e_shoulder_pan_joint']}</param>
+                </state_interface>
+                <state_interface name="velocity"/>
+                <state_interface name="effort"/>
+            </joint>
+            <joint name="410_ur5e_shoulder_lift_joint">
+                <command_interface name="position"/>
+                <command_interface name="velocity"/>
+                <command_interface name="effort"/>
+                <state_interface name="position">
+                  <param name="initial_value">${initial_positions['410_ur5e_shoulder_lift_joint']}</param>
+                </state_interface>
+                <state_interface name="velocity"/>
+                <state_interface name="effort"/>
+            </joint>
+            <joint name="410_ur5e_elbow_joint">
+                <command_interface name="position"/>
+                <command_interface name="velocity"/>
+                <command_interface name="effort"/>
+                <state_interface name="position">
+                  <param name="initial_value">${initial_positions['410_ur5e_elbow_joint']}</param>
+                </state_interface>
+                <state_interface name="velocity"/>
+                <state_interface name="effort"/>
+            </joint>
+            <joint name="410_ur5e_wrist_1_joint">
+                <command_interface name="position"/>
+                <command_interface name="velocity"/>
+                <command_interface name="effort"/>
+                <state_interface name="position">
+                  <param name="initial_value">${initial_positions['410_ur5e_wrist_1_joint']}</param>
+                </state_interface>
+                <state_interface name="velocity"/>
+                <state_interface name="effort"/>
+            </joint>
+            <joint name="410_ur5e_wrist_2_joint">
+                <command_interface name="position"/>
+                <command_interface name="velocity"/>
+                <command_interface name="effort"/>
+                <state_interface name="position">
+                  <param name="initial_value">${initial_positions['410_ur5e_wrist_2_joint']}</param>
+                </state_interface>
+                <state_interface name="velocity"/>
+                <state_interface name="effort"/>
+            </joint>
+            <joint name="410_ur5e_wrist_3_joint">
+                <command_interface name="position"/>
+                <command_interface name="velocity"/>
+                <command_interface name="effort"/>
+                <state_interface name="position">
+                  <param name="initial_value">${initial_positions['410_ur5e_wrist_3_joint']}</param>
+                </state_interface>
+                <state_interface name="velocity"/>
+                <state_interface name="effort"/>
+            </joint>
         </ros2_control>
     </xacro:macro>

File: src/Universal_Robots_ROS2_Tutorials/my_robot_cell/my_robot_cell_control/urdf/my_robot_cell_controlled.urdf.xacro (robot description, xacro)
@@ -3,8 +3,8 @@
   <!--First, include the macro from our custom description-->
   <xacro:include filename="$(find my_robot_cell_description)/urdf/my_robot_cell_macro.xacro"/>
+  <!--The driver already provides a control tag for the UR arm, we can directly include-->
+  <xacro:include filename="$(find ur_robot_driver)/urdf/ur.ros2_control.xacro"/>
   <xacro:include filename="$(find my_robot_cell_description)/urdf/table.xacro"/>
   <xacro:include filename="$(find my_robot_cell_description)/urdf/safety_wall.xacro"/>
-  <!--The driver already provides a control tag for the UR arm, we can directly include-->
-  <xacro:include filename="$(find ur_robot_driver)/urdf/ur.ros2_control.xacro"/>
   <!--We need to specify the arguments used for parametrizing our description-->
   <xacro:arg name="ur_type" default="ur5e"/>
@@ -13,5 +13,6 @@
   <xacro:arg name="physical_parameters_file" default="$(find ur_description)/config/$(arg ur_type)/physical_parameters.yaml"/>
   <xacro:arg name="visual_parameters_file" default="$(find ur_description)/config/$(arg ur_type)/visual_parameters.yaml"/>
-  <xacro:arg name="robot_ip" default="0.0.0.0"/>
+  <xacro:arg name="robot_409_ip" default="192.168.1.100"/>
+  <xacro:arg name="robot_410_ip" default="192.168.1.103"/>
   <xacro:arg name="headless_mode" default="false" />
   <xacro:arg name="ur_script_filename" default="$(find ur_client_library)/resources/external_control.urscript"/>
@@ -29,7 +30,7 @@
   <!--Create the scene description including the robot-->
   <xacro:my_robot_cell
+    prefix="409_"
     parent="world"
     ur_type="$(arg ur_type)"
-    prefix="409"
     joint_limits_parameters_file="$(arg joint_limit_parameters_file)"
     kinematics_parameters_file="$(arg kinematics_parameters_file)"
@@ -41,8 +42,8 @@
   <!--Create the control tag for the UR robot-->
   <xacro:ur_ros2_control
-    name="$(arg ur_type)"
+    name="409_ur5e"
     tf_prefix="409_$(arg ur_type)_"
     kinematics_parameters_file="$(arg kinematics_parameters_file)"
-    robot_ip="$(arg robot_ip)"
+    robot_ip="$(arg robot_409_ip)"
     script_filename="$(arg ur_script_filename)"
     output_recipe_filename="$(arg ur_output_recipe_filename)"
@@ -51,4 +52,36 @@
     mock_sensor_commands="$(arg mock_sensor_commands)"
     headless_mode="$(arg headless_mode)"
+    reverse_port="50001"
+    script_sender_port="50002"
+    script_command_port="50004"
+    trajectory_port="50003"
+  />
+  <xacro:my_robot_cell
+    prefix="410_"
+    parent="world"
+    ur_type="$(arg ur_type)"
+    joint_limits_parameters_file="$(arg joint_limit_parameters_file)"
+    kinematics_parameters_file="$(arg kinematics_parameters_file)"
+    physical_parameters_file="$(arg physical_parameters_file)"
+    visual_parameters_file="$(arg visual_parameters_file)"
+>
+    <!-- Change position so it's not overlapping with first robot -->
+    <origin xyz="0 0 1" rpy="0 0 0" />
+</xacro:my_robot_cell>
+  <xacro:ur_ros2_control
+    name="410_ur5e"
+    tf_prefix="410_$(arg ur_type)_"
+    kinematics_parameters_file="$(arg kinematics_parameters_file)"
+    robot_ip="$(arg robot_410_ip)"
+    script_filename="$(arg ur_script_filename)"
+    output_recipe_filename="$(arg ur_output_recipe_filename)"
+    input_recipe_filename="$(arg ur_input_recipe_filename)"
+    use_mock_hardware="$(arg use_mock_hardware)"
+    mock_sensor_commands="$(arg mock_sensor_commands)"
+    headless_mode="$(arg headless_mode)"
+    reverse_port="50005"
+    script_sender_port="50006"
+    script_command_port="50008"
+    trajectory_port="50007"
   />
   <!--If you had more controlled devices in your description, e.g. a gripper, you can add another ros2_control tag here-->

File: src/Universal_Robots_ROS2_Tutorials/my_robot_cell/my_robot_cell_description/urdf/box.xacro (robot description, xacro)
@@ -1,11 +1,11 @@
 <?xml version="1.0"?>
 <robot xmlns:xacro="http://ros.org/wiki/xacro">
-  <xacro:macro name="box" params="parent prefix *origin">
-    <joint name="${prefix}_box_joint" type="fixed">
-      <parent link="${prefix}_ur5e_tool0" />
-      <child link="${prefix}_box" />
+  <xacro:macro name="box" params="parent *origin">
+    <joint name="${prefix}box_joint" type="fixed">
+      <parent link="${prefix}ur5e_tool0" />
+      <child link="${prefix}box" />
       <origin rpy="0 0 0" xyz="0 0 0.16"/>
     </joint>
-    <link name="${prefix}_box">
+    <link name="${prefix}box">
       <visual>
         <geometry>

File: src/Universal_Robots_ROS2_Tutorials/my_robot_cell/my_robot_cell_description/urdf/my_robot_cell.urdf.xacro (robot description, xacro)
@@ -19,6 +19,17 @@
   <xacro:my_robot_cell
     parent="world"
+    prefix="409_"
     ur_type="$(arg ur_type)"
-    prefix="409"
+    joint_limits_parameters_file="$(arg joint_limits_parameters_file)"
+    kinematics_parameters_file="$(arg kinematics_parameters_file)"
+    physical_parameters_file="$(arg physical_parameters_file)"
+    visual_parameters_file="$(arg visual_parameters_file)"
+    >
+      <origin xyz="0 0 0" rpy="0 0 0" />
+  </xacro:my_robot_cell>
+  <xacro:my_robot_cell
+    parent="world"
+    prefix="410_"
+    ur_type="$(arg ur_type)"
     joint_limits_parameters_file="$(arg joint_limits_parameters_file)"
     kinematics_parameters_file="$(arg kinematics_parameters_file)"

File: src/Universal_Robots_ROS2_Tutorials/my_robot_cell/my_robot_cell_description/urdf/my_robot_cell_macro.xacro (robot description, xacro)
@@ -7,6 +7,6 @@
     parent
     *origin
+    prefix
     ur_type
-    prefix
     joint_limits_parameters_file
     kinematics_parameters_file
@@ -14,15 +14,15 @@
     visual_parameters_file
     ">
-    <link name="${prefix}_robot_mount"/>
-    <joint name="${prefix}_base_to_robot_mount" type="fixed">
-      <parent link="${prefix}_robot_base_plate"/>
-      <child link="${prefix}_robot_mount"/>
+    <link name="${prefix}robot_mount"/>
+    <joint name="${prefix}base_to_robot_mount" type="fixed">
+      <parent link="${prefix}robot_base_plate"/>
+      <child link="${prefix}robot_mount"/>
       <origin xyz="0 0 0" rpy="0 0 ${pi}" />
     </joint>
     <!--This will create the specific robot-->
     <xacro:ur_robot
-      name="${prefix}_${ur_type}"
-      tf_prefix="${prefix}_${ur_type}_"
-      parent="${prefix}_robot_mount"
+      name="${prefix}${ur_type}"
+      tf_prefix="${prefix}${ur_type}_"
+      parent="${prefix}robot_mount"
       joint_limits_parameters_file="${joint_limits_parameters_file}"
       kinematics_parameters_file="${kinematics_parameters_file}"
@@ -32,5 +32,5 @@
       <origin xyz="0 0 0" rpy="0 0 0" />
     </xacro:ur_robot>
-    <xacro:box parent="${prefix}_ur5e_tool0" prefix="${prefix}">
+    <xacro:box parent="${prefix}ur5e_tool0">
       <origin xyz="0 0 0.1" rpy="0 0 0"/>
     </xacro:box>

File: src/Universal_Robots_ROS2_Tutorials/my_robot_cell/my_robot_cell_description/urdf/table.xacro (robot description, xacro)
@@ -3,5 +3,5 @@
   <xacro:macro name="table" params="parent *origin">
     <joint name="table_base_joint" type="fixed">
-      <parent link="${parent}" />
+      <parent link="world" />
       <child link="table" />
       <origin rpy="0 0 0" xyz="0 0 0.9"/>
