Commit message: DnDSRC

File: src/Universal_Robots_ROS2_Tutorials/my_robot_cell/my_robot_cell_control/urdf/my_robot_cell_controlled.urdf.xacro (robot description, xacro)
@@ -28,5 +28,5 @@
     visual_parameters_file="$(arg visual_parameters_file)"
   >
-    <origin xyz="0 0 0.9" rpy="0 0 0" />
+    <origin xyz="0 0 1" rpy="0 0 0" />
   </xacro:my_robot_cell>
   <!--Create the control tag for the UR robot-->

File: src/Universal_Robots_ROS2_Tutorials/my_robot_cell/my_robot_cell_description/urdf/my_robot_cell.urdf.xacro (robot description, xacro)
@@ -17,5 +17,5 @@
     visual_parameters_file="$(arg visual_parameters_file)"
     >
-      <origin xyz="0 0 0" rpy="0 0 1" />
+      <origin xyz="0 0 0" rpy="0 0 0" />
   </xacro:my_robot_cell>
 </robot>

File: src/Universal_Robots_ROS2_Tutorials/my_robot_cell/my_robot_cell_description/urdf/my_robot_cell_macro.xacro (robot description, xacro)
@@ -4,6 +4,6 @@
   <xacro:include filename="$(find my_robot_cell_description)/urdf/safety_wall.xacro"/>
   <xacro:include filename="$(find my_robot_cell_description)/urdf/table.xacro"/>
+  <xacro:include filename="$(find my_robot_cell_description)/urdf/box.xacro"/>
   <xacro:include filename="$(find my_robot_cell_description)/urdf/2fg7_gripper/urdf/onrobot_2fg7_gripper.urdf.xacro"/>
-  <xacro:include filename="$(find my_robot_cell_description)/urdf/box.xacro"/>
   <xacro:macro name="my_robot_cell" params="
     parent
@@ -42,6 +42,6 @@
       <origin xyz="0 0 0.1" rpy="0 0 0"/>
     </xacro:box>
-    <!--xacro:onrobot_2fg7_gripper prefix="onrobot_2fg7_gripper" parent ="ur5e_tool0">
-      <origin rpy="0 4.71239 0" xyz="0 0 0"/>
+    <!--xacro:onrobot_2fg7_gripper prefix= "onrobot_2fg7_gripper" parent="ur5e_tool0">
+      <origin yxz="0 0 0" rpy="0 4.71239 0"/>
     </xacro:onrobot_2fg7_gripper-->
   </xacro:macro>

Commit message: with one robot, everything in the urdf.xacro working

File: src/Universal_Robots_ROS2_Tutorials/my_robot_cell/my_robot_cell_control/urdf/my_robot_cell_controlled.urdf.xacro (robot description, xacro)
@@ -5,4 +5,6 @@
   <!--The driver already provides a control tag for the UR arm, we can directly include-->
   <xacro:include filename="$(find ur_robot_driver)/urdf/ur.ros2_control.xacro"/>
+  <xacro:include filename="$(find my_robot_cell_description)/urdf/safety_wall.xacro"/>
+  <xacro:include filename="$(find my_robot_cell_description)/urdf/table.xacro"/>
   <!--We need to specify the arguments used for parametrizing our description-->
   <xacro:arg name="ur_type" default="ur5e"/>
@@ -20,4 +22,10 @@
   <link name="world" />
   <!--Create the scene description including the robot-->
+  <xacro:safety_wall parent="world">
+    <origin rpy="0 0 0" xyz="0 0 0"/>
+  </xacro:safety_wall>
+  <xacro:table parent="world">
+    <origin rpy="0 0 0" xyz="0 -0 0.9"/>
+  </xacro:table>
   <xacro:my_robot_cell
     parent="world"

File: src/Universal_Robots_ROS2_Tutorials/my_robot_cell/my_robot_cell_description/urdf/my_robot_cell.urdf.xacro (robot description, xacro)
@@ -2,4 +2,6 @@
 <robot name="my_robot_cell" xmlns:xacro="http://ros.org/wiki/xacro">
   <xacro:include filename="$(find my_robot_cell_description)/urdf/my_robot_cell_macro.xacro"/>
+  <xacro:include filename="$(find my_robot_cell_description)/urdf/safety_wall.xacro"/>
+  <xacro:include filename="$(find my_robot_cell_description)/urdf/table.xacro"/>
   <xacro:arg name="ur_type" default="ur5e"/>
   <xacro:arg name="joint_limits_parameters_file" default="$(find ur_description)/config/$(arg ur_type)/joint_limits.yaml"/>
@@ -9,7 +11,14 @@
   <link name="world"/>
   <!--This will create the scene where the robot is located in-->
+  <xacro:safety_wall parent="world">
+    <origin rpy="0 0 0" xyz="0 0 0"/>
+  </xacro:safety_wall>
+  <xacro:table parent="world">
+    <origin rpy="0 0 0" xyz="0 -0 0.9"/>
+  </xacro:table>
   <xacro:my_robot_cell
     parent="world"
     ur_type="$(arg ur_type)"
+    prefix="409"
     joint_limits_parameters_file="$(arg joint_limits_parameters_file)"
     kinematics_parameters_file="$(arg kinematics_parameters_file)"

File: src/Universal_Robots_ROS2_Tutorials/my_robot_cell/my_robot_cell_description/urdf/my_robot_cell_macro.xacro (robot description, xacro)
@@ -2,6 +2,4 @@
 <robot xmlns:xacro="http://ros.org/wiki/xacro">
   <xacro:include filename="$(find ur_description)/urdf/ur_macro.xacro"/>
-  <xacro:include filename="$(find my_robot_cell_description)/urdf/safety_wall.xacro"/>
-  <xacro:include filename="$(find my_robot_cell_description)/urdf/table.xacro"/>
   <xacro:include filename="$(find my_robot_cell_description)/urdf/box.xacro"/>
   <xacro:include filename="$(find my_robot_cell_description)/urdf/2fg7_gripper/urdf/onrobot_2fg7_gripper.urdf.xacro"/>
@@ -15,13 +13,7 @@
     visual_parameters_file
     ">
-    <xacro:table parent="${parent}">
-      <origin rpy="0 0 0" xyz="0 -0 0.9"/>
-    </xacro:table>
-    <xacro:safety_wall parent="${parent}">
-      <origin rpy="0 0 0" xyz="0 0 0"/>
-    </xacro:safety_wall>
     <link name="robot_mount"/>
-    <joint name="base_to_robot_mount_409" type="fixed">
-      <parent link="robot_base_plate_409"/>
+    <joint name="base_to_robot_mount" type="fixed">
+      <parent link="robot_base_plate"/>
       <child link="robot_mount"/>
       <origin xyz="0 0 0" rpy="0 0 ${pi}" />

File: src/Universal_Robots_ROS2_Tutorials/my_robot_cell/my_robot_cell_description/urdf/table.xacro (robot description, xacro)
@@ -32,10 +32,10 @@
     </link>
     <!--For Robot 409-->
-    <joint name="robot_base_plate_joint_409" type="fixed">
+    <joint name="robot_base_plate_joint" type="fixed">
       <parent link="table" />
-      <child link="robot_base_plate_409"/>
+      <child link="robot_base_plate"/>
       <origin rpy="0 0 0" xyz="-0.52 0.32 0.02"/>
     </joint>
-    <link name="robot_base_plate_409">
+    <link name="robot_base_plate">
       <visual>
         <geometry>

Commit message: same and possible to load in moveit setup assistant!

File: src/Universal_Robots_ROS2_Tutorials/my_robot_cell/my_robot_cell_control/urdf/my_robot_cell_controlled.urdf.xacro (robot description, xacro)
@@ -3,4 +3,6 @@
   <!--First, include the macro from our custom description-->
   <xacro:include filename="$(find my_robot_cell_description)/urdf/my_robot_cell_macro.xacro"/>
+  <xacro:include filename="$(find my_robot_cell_description)/urdf/table.xacro"/>
+  <xacro:include filename="$(find my_robot_cell_description)/urdf/safety_wall.xacro"/>
   <!--The driver already provides a control tag for the UR arm, we can directly include-->
   <xacro:include filename="$(find ur_robot_driver)/urdf/ur.ros2_control.xacro"/>
@@ -19,4 +21,10 @@
   <xacro:arg name="mock_sensor_commands" default="false" />
   <link name="world" />
+  <xacro:table parent="world">
+    <origin rpy="0 0 0" xyz="0 -0 0.9"/>
+  </xacro:table>
+  <xacro:safety_wall parent="world">
+    <origin rpy="0 0 0" xyz="0 0 0"/>
+  </xacro:safety_wall>
   <!--Create the scene description including the robot-->
   <xacro:my_robot_cell

File: src/Universal_Robots_ROS2_Tutorials/my_robot_cell/my_robot_cell_description/urdf/my_robot_cell.urdf.xacro (robot description, xacro)
@@ -2,4 +2,6 @@
 <robot name="my_robot_cell" xmlns:xacro="http://ros.org/wiki/xacro">
   <xacro:include filename="$(find my_robot_cell_description)/urdf/my_robot_cell_macro.xacro"/>
+  <xacro:include filename="$(find my_robot_cell_description)/urdf/table.xacro"/>
+  <xacro:include filename="$(find my_robot_cell_description)/urdf/safety_wall.xacro"/>
   <xacro:arg name="ur_type" default="ur5e"/>
   <xacro:arg name="joint_limits_parameters_file" default="$(find ur_description)/config/$(arg ur_type)/joint_limits.yaml"/>
@@ -9,4 +11,10 @@
   <link name="world"/>
   <!--This will create the scene where the robot is located in-->
+  <xacro:table parent="world">
+    <origin rpy="0 0 0" xyz="0 -0 0.9"/>
+  </xacro:table>
+  <xacro:safety_wall parent="world">
+    <origin rpy="0 0 0" xyz="0 0 0"/>
+  </xacro:safety_wall>
   <xacro:my_robot_cell
     parent="world"

File: src/Universal_Robots_ROS2_Tutorials/my_robot_cell/my_robot_cell_description/urdf/my_robot_cell_macro.xacro (robot description, xacro)
@@ -2,6 +2,4 @@
 <robot xmlns:xacro="http://ros.org/wiki/xacro">
   <xacro:include filename="$(find ur_description)/urdf/ur_macro.xacro"/>
-  <xacro:include filename="$(find my_robot_cell_description)/urdf/safety_wall.xacro"/>
-  <xacro:include filename="$(find my_robot_cell_description)/urdf/table.xacro"/>
   <xacro:include filename="$(find my_robot_cell_description)/urdf/box.xacro"/>
   <xacro:include filename="$(find my_robot_cell_description)/urdf/2fg7_gripper/urdf/onrobot_2fg7_gripper.urdf.xacro"/>
@@ -15,10 +13,4 @@
     visual_parameters_file
     ">
-    <xacro:table parent="${parent}">
-      <origin rpy="0 0 0" xyz="0 -0 0.9"/>
-    </xacro:table>
-    <xacro:safety_wall parent="${parent}">
-      <origin rpy="0 0 0" xyz="0 0 0"/>
-    </xacro:safety_wall>
     <link name="robot_mount"/>
     <joint name="base_to_robot_mount" type="fixed">

Commit message: with one robot turned pi/2

File: src/Universal_Robots_ROS2_Tutorials/my_robot_cell/my_robot_cell_control/urdf/my_robot_cell_controlled.urdf.xacro (robot description, xacro)
@@ -30,4 +30,5 @@
   <!--Create the scene description including the robot-->
   <xacro:my_robot_cell
+    angle="${pi}"
     prefix="409_"
     parent="world"
@@ -58,4 +59,5 @@
   />
   <xacro:my_robot_cell
+    angle="${pi/2}"
     prefix="410_"
     parent="world"

File: src/Universal_Robots_ROS2_Tutorials/my_robot_cell/my_robot_cell_description/urdf/my_robot_cell.urdf.xacro (robot description, xacro)
@@ -18,4 +18,5 @@
   </xacro:safety_wall>
   <xacro:my_robot_cell
+    angle="${pi}"
     parent="world"
     prefix="409_"
@@ -29,4 +30,5 @@
   </xacro:my_robot_cell>
   <xacro:my_robot_cell
+    angle="${pi/2}"
     parent="world"
     prefix="410_"

File: src/Universal_Robots_ROS2_Tutorials/my_robot_cell/my_robot_cell_description/urdf/my_robot_cell_macro.xacro (robot description, xacro)
@@ -5,4 +5,5 @@
   <xacro:include filename="$(find my_robot_cell_description)/urdf/2fg7_gripper/urdf/onrobot_2fg7_gripper.urdf.xacro"/>
   <xacro:macro name="my_robot_cell" params="
+    angle
     parent
     *origin
@@ -18,5 +19,5 @@
       <parent link="${prefix}robot_base_plate"/>
       <child link="${prefix}robot_mount"/>
-      <origin xyz="0 0 0" rpy="0 0 ${pi}" />
+      <origin xyz="0 0 0" rpy="0 0 ${angle}" />
     </joint>
     <!--This will create the specific robot-->

Commit message: motion planning somehow works

File: src/Universal_Robots_ROS2_Tutorials/my_robot_cell/my_robot_cell_control/urdf/my_robot_cell_controlled.urdf.xacro (robot description, xacro)
@@ -30,5 +30,5 @@
   <!--Create the scene description including the robot-->
   <xacro:my_robot_cell
-    angle="${pi}"
+    rotation="0 0 0"
     prefix="409_"
     parent="world"
@@ -59,5 +59,5 @@
   />
   <xacro:my_robot_cell
-    angle="${pi/2}"
+    rotation="0 0 -${pi/2}"
     prefix="410_"
     parent="world"

File: src/Universal_Robots_ROS2_Tutorials/my_robot_cell/my_robot_cell_description/urdf/my_robot_cell.urdf.xacro (robot description, xacro)
@@ -18,5 +18,5 @@
   </xacro:safety_wall>
   <xacro:my_robot_cell
-    angle="${pi}"
+    rotation="0 0 0"
     parent="world"
     prefix="409_"
@@ -30,5 +30,5 @@
   </xacro:my_robot_cell>
   <xacro:my_robot_cell
-    angle="${pi/2}"
+    rotation="0 0  -${pi/2}"
     parent="world"
     prefix="410_"

File: src/Universal_Robots_ROS2_Tutorials/my_robot_cell/my_robot_cell_description/urdf/my_robot_cell_macro.xacro (robot description, xacro)
@@ -5,6 +5,6 @@
   <xacro:include filename="$(find my_robot_cell_description)/urdf/2fg7_gripper/urdf/onrobot_2fg7_gripper.urdf.xacro"/>
   <xacro:macro name="my_robot_cell" params="
-    angle
     parent
+    rotation
     *origin
     prefix
@@ -19,5 +19,5 @@
       <parent link="${prefix}robot_base_plate"/>
       <child link="${prefix}robot_mount"/>
-      <origin xyz="0 0 0" rpy="0 0 ${angle}" />
+      <origin xyz="0 0 0" rpy="0 0 ${pi}" />
     </joint>
     <!--This will create the specific robot-->
@@ -31,5 +31,5 @@
       visual_parameters_file="${visual_parameters_file}"
     >
-      <origin xyz="0 0 0" rpy="0 0 0" />
+      <origin xyz="0 0 0" rpy="${rotation}" />
     </xacro:ur_robot>
     <xacro:box parent="${prefix}ur5e_tool0">
